File: production/ecad/Tubender PCB/untitled.kicad_sch (KiCad schematic)
At the start: 0 parts

Commit message: added name on power sheet
Other:
- note added: "Nikolas Varga"
Changed lines of the file:
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@@
-(kicad_sch (version 20230121) (generator eeschema)
-  (paper "A4")
+(kicad_sch
+	(version 20231120)
+	(generator "eeschema")
+	(generator_version "8.0")
+	(paper "A4")
+	(text "Nikolas Varga"
+		(exclude_from_sim no)
+		(at 194.056 173.482 0)
+		(effects
+			(font
+				(size 1.27 1.27)
+			)
+		)
+	)
 )
