File: production/ecad/Tubender PCB/untitled.kicad_sch (KiCad schematic)
At the start: 0 parts

Commit message: added 3.3V buck IC symbol and changed power sheet directory
Other:
- note added: "Nik"
Changed lines of the file:
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@@
 	(generator_version "8.0")
 	(paper "A4")
+	(text "Nik"
+		(exclude_from_sim no)
+		(at 199.644 189.484 0)
+		(effects
+			(font
+				(size 1.27 1.27)
+			)
+		)
+	)
 )

Commit message: Added 3V3 buck circuitry to main branch, added 3V3 label
Other:
- note removed: "Nik"
Changed lines of the file:
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@@
 	(generator_version "8.0")
 	(paper "A4")
-	(text "Nik"
-		(exclude_from_sim no)
-		(at 199.644 189.484 0)
-		(effects
-			(font
-				(size 1.27 1.27)
-			)
-		)
-	)
 )
