File: production/ecad/Tubender PCB/untitled.kicad_sch (KiCad schematic)
At the start: 0 parts

Commit message: First MCU Edit
Parts:
- added U4: ESP32-S3, Package_DFN_QFN:QFN-56-1EP_7x7mm_P0.4mm_EP4x4mm, symbol MCU_Espressif:ESP32-S3
Connections:
- new net: U4.2 (VDD3P3), U4.3 (VDD3P3)
- new net: U4.55 (VDDA), U4.56 (VDDA)
- new net CHUCK_CLAMP_DIR+: U4.42 (GPIO37)
- new net CHUCK_CLAMP_ENA+: U4.41 (GPIO36)
- new net CHUCK_CLAMP_PUL+: U4.40 (GPIO35)
- new net DIE_CLAMP_DIR+: U4.19 (GPIO14)
- new net DIE_CLAMP_ENA+: U4.18 (GPIO13)
- new net DIE_CLAMP_PUL+: U4.17 (GPIO12)
