File: production/ecad/Tubender PCB/microcontroller.kicad_sch (KiCad schematic)
At the start: 0 parts

Commit message: Add microcontroller to control schematic
Parts:
- added U1: ESP32-WROOM-E, PCM_Espressif:ESP32-WROOM-32E, symbol PCM_Espressif:ESP32-WROOM-E
Connections:
- new net: U1.1 (GND), U1.15 (GND), U1.38 (GND)
Changed lines of the file:
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@@
 	(generator_version "8.0")
 	(paper "A4")
+	(symbol
+		(lib_id "PCM_Espressif:ESP32-WROOM-E")
+		(at 137.16 85.09 0)
+		(unit 1)
+		(exclude_from_sim no)
+		(in_bom yes)
+		(on_board yes)
+		(dnp no)
+		(fields_autoplaced yes)
+		(property "Reference" "U1"
+			(at 139.3541 57.15 0)
+			(effects
+				(font
+					(size 1.27 1.27)
+				)
+				(justify left)
+			)
+		)
+		(property "Value" "ESP32-WROOM-E"
+			(at 139.3541 59.69 0)
+			(effects
+				(font
+					(size 1.27 1.27)
+				)
+				(justify left)
+			)
+		)
+		(property "Footprint" "PCM_Espressif:ESP32-WROOM-32E"
+			(at 137.16 120.65 0)
+			(effects
+				(font
+					(size 1.27 1.27)
+				)
+				(hide yes)
+			)
+		)
+		(property "Datasheet" "https://www.espressif.com/sites/default/files/documentation/esp32-wroom-32e_esp32-wroom-32ue_datasheet_en.pdf"
+			(at 137.16 123.19 0)
+			(effects
+				(font
+					(size 1.27 1.27)
+				)
+				(hide yes)
+			)
+		)
+		(property "Description" "ESP32-WROOM-32E integrates ESP32-D0WD-V3, with higher stability and safety performance."
+			(at 137.16 85.09 0)
+			(effects
+				(font
+					(size 1.27 1.27)
+				)
+				(hide yes)
+			)
+		)
+		(pin "25"
+		)
+		(pin "10"
+		)
+		(pin "39"
+		)
+		(pin "30"
+		)
+		(pin "12"
+		)
+		(pin "13"
+		)
+		(pin "31"
+		)
+		(pin "28"
+		)
+		(pin "38"
+		)
+		(pin "2"
+		)
+		(pin "35"
+		)
+		(pin "26"
+		)
+		(pin "33"
+		)
+		(pin "11"
+		)
+		(pin "36"
+		)
+		(pin "7"
+		)
+		(pin "6"
+		)
+		(pin "27"
+		)
+		(pin "15"
+		)
+		(pin "8"
+		)
+		(pin "9"
+		)
+		(pin "16"
+		)
+		(pin "29"
+		)
+		(pin "1"
+		)
+		(pin "14"
+		)
+		(pin "24"
+		)
+		(pin "4"
+		)
+		(pin "23"
+		)
+		(pin "3"
+		)
+		(pin "5"
+		)
+		(pin "37"
+		)
+		(pin "34"
+		)
+		(instances
+			(project ""
+				(path "/3e1aedd0-6089-4edb-92c7-0c31da2e7927/65adf537-572f-4850-8052-0180b0042e43/26fa3857-1fd4-4f90-a473-c468ba375965"
+					(reference "U1")
+					(unit 1)
+				)
+			)
+		)
+	)
 )
