File: production/ecad/Tubender PCB/temp.kicad_sch (KiCad schematic)
At the start: 6 parts, among them IC7 SN74LVC1G29DCTR, U7 74HC595, U8 CD4051BE, U9 CD4051BE

Commit message: final for rev 1
Parts:
- removed C12: 0.1uF, symbol Device:C
- removed DS2: BC56-12EWA, DIPS1524W50P254L3760H835Q12N, symbol SamacSys_Parts:BC56-12EWA
- removed IC7: SN74LVC1G29DCTR, SOP65P400X130-8N, symbol SamacSys_Parts:SN74LVC1G29DCTR
- removed U7: 74HC595, symbol 74xx:74HC595
- removed U8, U9: CD4051BE, CD4051BE:DIP794W45P254L1969H508Q16, symbol CD4051BE:CD4051BE
Connections:
- no-connect marks 4 -> 0
