File: production/ecad/Tubender PCB/user_interface.kicad_sch (KiCad schematic)
At the start: 97 parts, among them IC1 74HC4050D, IC2 RA8875L3N, IC3 CD4051BM96, IC4 CD4051BM96, J12 640387-2, J15 640387-2, J16 640387-2, J17 640387-2, J18 640387-2, J19 640387-2, J20 640387-2, J21 640387-2, J22 640387-2, J23 640387-2, J24 640387-2, J25 640387-2, J26 640387-2, J27 640387-2, J28 640387-2, J29 1-640387-0, J31 640387-5, J7 4-1734592-0, U11 SN74AHC1G125DBVR, Y1 ABM8-20.000MHz-10-B1U-T

Commit message: working on mcu layout
Parts:
- IC1: footprint footprints:SOT109-1_NXP -> ${KIPRJMOD}:SOT109-1_NXP
- IC2: footprint footprints:QFP40P1600X1600X160-128N -> ${KIPRJMOD}:QFP40P1600X1600X160-128N
- IC3, IC4: footprint footprints:SOIC127P600X175-16N -> ${KIPRJMOD}:SOIC127P600X175-16N
- J7: footprint footprints:TE_4-1734592-0 -> ${KIPRJMOD}:TE_4-1734592-0
- TP14, TP15, TP16, TP17, TP18, TP19, TP20, TP21, TP22, TP23, TP24, TP25, TP26, TP27: footprint 5006:KEYSTONE_5006 -> ${KIPRJMOD}:KEYSTONE_5006
Changed lines of the file:
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@@
 			)
 		)
-		(property "Footprint" "5006:KEYSTONE_5006"
+		(property "Footprint" "${KIPRJMOD}:KEYSTONE_5006"
 			(at 129.54 128.27 0)
 			(effects
@@
 			)
 		)
-		(property "Footprint" "5006:KEYSTONE_5006"
+		(property "Footprint" "${KIPRJMOD}:KEYSTONE_5006"
 			(at 125.73 124.46 0)
 			(effects
@@
 			)
 		)
-		(property "Footprint" "5006:KEYSTONE_5006"
+		(property "Footprint" "${KIPRJMOD}:KEYSTONE_5006"
 			(at 153.67 140.97 0)
 			(effects
@@
 			)
 		)
-		(property "Footprint" "5006:KEYSTONE_5006"
+		(property "Footprint" "${KIPRJMOD}:KEYSTONE_5006"
 			(at 128.27 147.32 0)
 			(effects
@@
 			)
 		)
-		(property "Footprint" "5006:KEYSTONE_5006"
+		(property "Footprint" "${KIPRJMOD}:KEYSTONE_5006"
 			(at 81.28 151.13 0)
 			(effects
@@
 			)
 		)
-		(property "Footprint" "footprints:SOIC127P600X175-16N"
+		(property "Footprint" "${KIPRJMOD}:SOIC127P600X175-16N"
 			(at 353.06 216.84 0)
 			(effects
@@
 			)
 		)
-		(property "Footprint" "5006:KEYSTONE_5006"
+		(property "Footprint" "${KIPRJMOD}:KEYSTONE_5006"
 			(at 146.05 138.43 0)
 			(effects
@@
 			)
 		)
-		(property "Footprint" "5006:KEYSTONE_5006"
+		(property "Footprint" "${KIPRJMOD}:KEYSTONE_5006"
 			(at 116.84 90.17 0)
 			(effects
@@
 			)
 		)
-		(property "Footprint" "5006:KEYSTONE_5006"
+		(property "Footprint" "${KIPRJMOD}:KEYSTONE_5006"
 			(at 124.46 151.13 0)
 			(effects
@@
 			)
 		)
-		(property "Footprint" "5006:KEYSTONE_5006"
+		(property "Footprint" "${KIPRJMOD}:KEYSTONE_5006"
 			(at 118.11 50.8 0)
 			(effects
@@
 			)
 		)
-		(property "Footprint" "5006:KEYSTONE_5006"
+		(property "Footprint" "${KIPRJMOD}:KEYSTONE_5006"
 			(at 88.9 52.07 0)
 			(effects
@@
 			)
 		)
-		(property "Footprint" "5006:KEYSTONE_5006"
+		(property "Footprint" "${KIPRJMOD}:KEYSTONE_5006"
 			(at 88.9 123.19 0)
 			(effects
@@
 			)
 		)
-		(property "Footprint" "footprints:SOT109-1_NXP"
+		(property "Footprint" "${KIPRJMOD}:SOT109-1_NXP"
 			(at 118.11 228.27 0)
 			(effects
@@
 			)
 		)
-		(property "Footprint" "footprints:QFP40P1600X1600X160-128N"
+		(property "Footprint" "${KIPRJMOD}:QFP40P1600X1600X160-128N"
 			(at 231.14 143.18 0)
 			(effects
@@
 			)
 		)
-		(property "Footprint" "5006:KEYSTONE_5006"
+		(property "Footprint" "${KIPRJMOD}:KEYSTONE_5006"
 			(at 86.36 129.54 0)
 			(effects
@@
 			)
 		)
-		(property "Footprint" "footprints:TE_4-1734592-0"
+		(property "Footprint" "${KIPRJMOD}:TE_4-1734592-0"
 			(at 44.45 144.45 0)
 			(effects
@@
 			)
 		)
-		(property "Footprint" "5006:KEYSTONE_5006"
+		(property "Footprint" "${KIPRJMOD}:KEYSTONE_5006"
 			(at 144.78 86.36 0)
 			(effects
@@
 			)
 		)
-		(property "Footprint" "footprints:SOIC127P600X175-16N"
+		(property "Footprint" "${KIPRJMOD}:SOIC127P600X175-16N"
 			(at 353.06 171.12 0)
 			(effects
@@
 			)
 		)
-		(property "Footprint" "5006:KEYSTONE_5006"
+		(property "Footprint" "${KIPRJMOD}:KEYSTONE_5006"
 			(at 88.9 102.87 0)
 			(effects
