File: production/ecad/Tubender PCB/Tubender PCB.kicad_pcb (KiCad board)
At the start: 2 copper layers, 253 parts, among them IC1 74HC4050D, IC2 RA8875L3N, IC3 CD4051BM96, IC4 CD4051BM96, J1 640387-2, J10 640387-2, J10 640387-5, J11 640387-8, J12 640387-2, J13 640387-5, J14 640387-3, J15 640387-2, J16 640387-2, J17 640387-2, J18 640387-2, J19 640387-2, J2 640387-5, J20 640387-2, J21 640387-2, J22 640387-2, J23 640387-2, J24 640387-2, J25 640387-2, J26 640387-2, J27 640387-2, J28 640387-2, J29 1-640387-0, J3 640387-5, J30 640387-2, J31 640387-5, J32 USB4110GFA, J33 640387-2, J34 640387-2, J35 640387-3, J37 640387-3, J4 640387-5, J5 640387-2, J5 640387-6, J6 640387-2, J6 640387-6, J7 4-1734592-0, J8 640387-3, J8 640387-6, J9 640387-3, J9 640387-5, Q1 AO3400A, Q2 AO3400A, U1 LMR36520FADDAR, U10 MCP23017-E_SO, U11 SN74AHC1G125DBVR, U12 LM5146RGYR, U13 LM5017SDX/NOPB, U2 ESP32-WROOM-32UE_M113EH6400UH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, U3 MCP23017-E_SO, U5 TPSM265R1V5SILR, U6 CP2102N-A02-GQFN28, Y1 ABM8-20.000MHz-10-B1U-T

Commit message: more traces
Routing:
- net 7-SEG_A0: track 0.00 -> 119.4 mm
- net 7-SEG_SER: track 0.00 -> 112.3 mm
- net 7-SEG_SRCLK: track 0.00 -> 94.0 mm
- net 7-SEG_RCLK: track 0.00 -> 91.5 mm
- net 7-SEG_OEb: track 0.00 -> 88.9 mm
- net BUTTON_3: track 326.9 -> 319.8 mm
Changed lines of the file:
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@@
+	)
+	(segment
+		(start 210.5 148.95)
+		(end 210.475 148.975)
+		(width 0.25)
+		(layer "F.Cu")
+		(net 15)
+	)
+	(segment
+		(start 66.75 220.25)
+		(end 64.25 217.75)
+		(width 0.25)
+		(layer "F.Cu")
+		(net 15)
+	)
+	(segment
+		(start 60.55 196.75)
+		(end 60.55 200.3325)
+		(width 0.25)
+		(layer "F.Cu")
+		(net 15)
+	)
+	(segment
+		(start 210.5 144.5)
+		(end 210.5 148.95)
+		(width 0.25)
+		(layer "F.Cu")
+		(net 15)
+	)
+	(segment
+		(start 285.3 144.54)
+		(end 271.79 144.54)
+		(width 0.25)
+		(layer "F.Cu")
+		(net 15)
+	)
+	(segment
+		(start 58.8 195)
+		(end 57.1625 195)
+		(width 0.25)
+		(layer "F.Cu")
+		(net 15)
+	)
+	(segment
+		(start 64.25 204.0325)
+		(end 60.5875 200.37)
+		(width 0.25)
+		(layer "F.Cu")
+		(net 15)
+	)
+	(segment
+		(start 60.55 200.3325)
+		(end 60.5875 200.37)
+		(width 0.25)
+		(layer "F.Cu")
+		(net 15)
+	)
+	(segment
+		(start 210.475 148.975)
+		(end 210.475 191.638604)
+		(width 0.25)
+		(layer "F.Cu")
+		(net 15)
+	)
+	(segment
+		(start 210.475 191.638604)
+		(end 206 196.113604)
+		(width 0.25)
+		(layer "F.Cu")
+		(net 15)
+	)
+	(segment
+		(start 206 196.113604)
+		(end 206 216.75)
+		(width 0.25)
+		(layer "F.Cu")
+		(net 15)
+	)
+	(segment
+		(start 206 216.75)
+		(end 202.5 220.25)
+		(width 0.25)
+		(layer "F.Cu")
+		(net 15)
+	)
+	(segment
+		(start 64.25 217.75)
+		(end 64.25 204.0325)
+		(width 0.25)
+		(layer "F.Cu")
+		(net 15)
 	)
 	(segment
 		(start 202.5 220.25)
 		(end 66.75 220.25)
-		(width 0.25)
-		(layer "F.Cu")
-		(net 15)
-	)
-	(segment
-		(start 206 196.113604)
-		(end 206 216.75)
-		(width 0.25)
-		(layer "F.Cu")
-		(net 15)
-	)
-	(segment
-		(start 205.75 144.25)
-		(end 210.475 148.975)
-		(width 0.25)
-		(layer "F.Cu")
-		(net 15)
-	)
-	(segment
-		(start 60.55 196.75)
-		(end 60.55 200.3325)
-		(width 0.25)
-		(layer "F.Cu")
-		(net 15)
-	)
-	(segment
-		(start 285.3 144.54)
-		(end 271.79 144.54)
-		(width 0.25)
-		(layer "F.Cu")
-		(net 15)
-	)
-	(segment
-		(start 58.8 195)
-		(end 57.1625 195)
-		(width 0.25)
-		(layer "F.Cu")
-		(net 15)
-	)
-	(segment
-		(start 60.55 200.3325)
-		(end 60.5875 200.37)
-		(width 0.25)
-		(layer "F.Cu")
-		(net 15)
-	)
-	(segment
-		(start 64.25 217.75)
-		(end 64.25 204.0325)
-		(width 0.25)
-		(layer "F.Cu")
-		(net 15)
-	)
-	(segment
-		(start 66.75 220.25)
-		(end 64.25 217.75)
-		(width 0.25)
-		(layer "F.Cu")
-		(net 15)
-	)
-	(segment
-		(start 206 216.75)
-		(end 202.5 220.25)
-		(width 0.25)
-		(layer "F.Cu")
-		(net 15)
-	)
-	(segment
-		(start 210.475 191.638604)
-		(end 206 196.113604)
-		(width 0.25)
-		(layer "F.Cu")
-		(net 15)
-	)
-	(segment
-		(start 210.475 148.975)
-		(end 210.475 191.638604)
-		(width 0.25)
-		(layer "F.Cu")
-		(net 15)
-	)
-	(segment
-		(start 64.25 204.0325)
-		(end 60.5875 200.37)
 		(width 0.25)
 		(layer "F.Cu")
@@
 	)
 	(via
-		(at 205.75 144.25)
+		(at 210.5 144.5)
 		(size 0.8)
 		(drill 0.4)
@@
 	)
 	(segment
-		(start 271.75 144.5)
-		(end 206 144.5)
-		(width 0.25)
-		(layer "B.Cu")
-		(net 15)
-	)
-	(segment
-		(start 206 144.5)
-		(end 205.75 144.25)
+		(start 210.5 144.5)
+		(end 271.75 144.5)
 		(width 0.25)
 		(layer "B.Cu")
@@
 	)
 	(segment
+		(start 221.864528 130.837375)
+		(end 175.0902 177.611703)
+		(width 0.25)
+		(layer "F.Cu")
+		(net 79)
+	)
+	(segment
+		(start 226.9575 130.837375)
+		(end 221.864528 130.837375)
+		(width 0.25)
+		(layer "F.Cu")
+		(net 79)
+	)
+	(segment
+		(start 175.0902 177.611703)
+		(end 175.0902 200.37)
+		(width 0.25)
+		(layer "F.Cu")
+		(net 79)
+	)
+	(segment
+		(start 175.25 203.25)
+		(end 184.0902 203.25)
+		(width 0.25)
+		(layer "F.Cu")
+		(net 80)
+	)
+	(segment
+		(start 226.9575 129.567375)
+		(end 222.498132 129.567375)
+		(width 0.25)
+		(layer "F.Cu")
+		(net 80)
+	)
+	(segment
+		(start 184.0902 203.25)
+		(end 186.9702 200.37)
+		(width 0.25)
+		(layer "F.Cu")
+		(net 80)
+	)
+	(segment
+		(start 173.25 178.815507)
+		(end 173.25 201.25)
+		(width 0.25)
+		(layer "F.Cu")
+		(net 80)
+	)
+	(segment
+		(start 173.25 201.25)
+		(end 175.25 203.25)
+		(width 0.25)
+		(layer "F.Cu")
+		(net 80)
+	)
+	(segment
+		(start 222.498132 129.567375)
+		(end 173.25 178.815507)
+		(width 0.25)
+		(layer "F.Cu")
+		(net 80)
+	)
+	(segment
+		(start 183.0102 170.964495)
+		(end 183.0102 200.37)
+		(width 0.25)
+		(layer "F.Cu")
+		(net 81)
+	)
+	(segment
+		(start 226.9575 133.377375)
+		(end 220.59732 133.377375)
+		(width 0.25)
+		(layer "F.Cu")
+		(net 81)
+	)
+	(segment
+		(start 220.59732 133.377375)
+		(end 183.0102 170.964495)
+		(width 0.25)
+		(layer "F.Cu")
+		(net 81)
+	)
+	(segment
+		(start 221.230924 132.107375)
+		(end 226.9575 132.107375)
+		(width 0.25)
+		(layer "F.Cu")
+		(net 82)
+	)
+	(segment
+		(start 179.0502 200.37)
+		(end 179.0502 174.288099)
+		(width 0.25)
+		(layer "F.Cu")
+		(net 82)
+	)
+	(segment
+		(start 179.0502 174.288099)
+		(end 221.230924 132.107375)
+		(width 0.25)
+		(layer "F.Cu")
+		(net 82)
+	)
+	(segment
 		(start 226.9575 127.027375)
 		(end 226.007501 127.027375)
@@
 	)
 	(segment
+		(start 175.063604 203.7)
+		(end 172.75 201.386396)
+		(width 0.25)
+		(layer "F.Cu")
+		(net 84)
+	)
+	(segment
+		(start 187.6002 203.7)
+		(end 175.063604 203.7)
+		(width 0.25)
+		(layer "F.Cu")
+		(net 84)
+	)
+	(segment
+		(start 225.671736 125.757375)
+		(end 226.9575 125.757375)
+		(width 0.25)
+		(layer "F.Cu")
+		(net 84)
+	)
+	(segment
+		(start 172.75 178.679111)
+		(end 225.671736 125.757375)
+		(width 0.25)
+		(layer "F.Cu")
+		(net 84)
+	)
+	(segment
+		(start 190.9302 200.37)
+		(end 187.6002 203.7)
+		(width 0.25)
+		(layer "F.Cu")
+		(net 84)
+	)
+	(segment
+		(start 172.75 201.386396)
+		(end 172.75 178.679111)
+		(width 0.25)
+		(layer "F.Cu")
+		(net 84)
+	)
+	(segment
