File: production/ecad/Tubender PCB/Tubender PCB.kicad_pcb (KiCad board)
At the start: 4 copper layers, 352.2 x 159.2 mm, 260 parts, among them IC1 74HC4050D, IC2 RA8875L3N, IC3 CD4051BM96, IC4 CD4051BM96, J1 640387-2, J10 640387-2, J10 640387-5, J11 640387-8, J12 640387-2, J13 640387-5, J14 640387-3, J15 640387-2, J16 640387-2, J17 640387-2, J18 640387-2, J19 640387-2, J2 640387-5, J20 640387-2, J21 640387-2, J22 640387-2, J23 640387-2, J24 640387-2, J25 640387-2, J26 640387-2, J27 640387-2, J28 640387-2, J29 1-640387-0, J3 640387-5, J30 640387-2, J31 640387-5, J32 USB4110GFA, J33 640387-2, J34 640387-2, J35 640387-3, J37 640387-3, J4 640387-5, J5 640387-2, J5 640387-6, J6 640387-2, J6 640387-6, J7 4-1734592-0, J8 640387-3, J8 640387-6, J9 640387-3, J9 640387-5, Q1 AO3400A, Q2 AO3400A, U1 LMR36520FADDAR, U10 MCP23017-E_SO, U11 SN74AHC1G125DBVR, U12 LM5146RGYR, U13 LM5017SDX/NOPB, U2 ESP32-WROOM-32UE_M113EH6400UH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, U3 MCP23017-E_SO, U5 TPSM265R1V5SILR, U6 CP2102N-A02-GQFN28, Y1 ABM8-20.000MHz-10-B1U-T

Commit message: Differential Pairs
Parts:
- moved R69 21.1 mm to (335.0, 99.5)
- moved R66 16.5 mm to (374.0, 81.7)
- moved C10 7.22 mm to (356.5, 91.5)
- moved D14 3.78 mm to (352.5, 93.8)
- moved C11 3.15 mm to (356.5, 95.0), turned to -90 degrees
- moved D13 2.99 mm to (354.5, 92.7), turned to -90 degrees
- moved D15 1.02 mm to (357.4, 99.7)
- moved C34 0.69 mm to (354.1, 100.0)
Connections:
- net Net-(J32-DN1) renamed /CONTROL/USB_DN
- net Net-(J32-DP1) renamed /CONTROL/USB_DP
Routing:
- net /CONTROL/USB_DP: track 21.1 -> 76.9 mm
- net /CONTROL/USB_DN: track 58.5 -> 76.7 mm, vias 2 -> 0
- net Net-(J32-CC1): track 13.5 -> 0.05 mm
- net Net-(J32-VBUS): track 26.4 -> 32.1 mm
- net GND: track 424.3 -> 429.2 mm, vias 86 -> 85
- net Net-(U6-VBUS): track 44.2 -> 40.2 mm, vias 0 -> 2
- net 48V: track 356.0 -> 355.9 mm, vias 11 -> 12
- net CHUCK_CLAMP_DIR+: vias 1 -> 0
- net ADVANCING_PUL+: vias 3 -> 2

Commit message: small changes and reducing errors
Parts:
- turned R_ILIM1 to 0 degrees
Connections:
- J7 pad 1: LEDK -> GND
Routing:
- net GND: track 429.2 -> 451.3 mm, vias 85 -> 86
- net Net-(Q_LO1-D): track 50.1 -> 59.5 mm
- net ESP_RXD0: track 109.4 -> 106.5 mm
- net ON/OFF: track 26.5 -> 28.0 mm
- net ADVANCING_DIR+: track 136.2 -> 135.2 mm
- net 3.3V: track 624.7 -> 625.6 mm
- net BENDING_LPWM: track 98.8 -> 99.6 mm
- net 48V: track 355.9 -> 356.7 mm

Commit message: got rid of all drc issues
Parts:
- added R84: 15k, Resistor_SMD:R_0805_2012Metric, F.Cu at (328.1, 96.5)
Connections:
- U12 pad 15: unconnected-(U12-EP-Pad15) -> GND
- U12 pad 21: unconnected-(U12-EP-Pad21) -> GND
- U12 pad 22: (no net) -> GND
- U12 pad 23: (no net) -> GND
- U12 pad 24: (no net) -> GND
- U12 pad 25: (no net) -> GND
- U5 pad V: (no net) -> GND
Routing:
- net Net-(J32-CC1): track 0.05 -> 16.9 mm, vias 0 -> 2
- net Net-(J14-Pad1): track 3.59 -> 17.3 mm
- net 48V: track 356.7 -> 366.1 mm, vias 12 -> 15
- net 24V: track 535.2 -> 541.8 mm, vias 8 -> 12
- net GND: track 451.3 -> 456.9 mm, vias 86 -> 87
- net 5V: track 621.0 -> 617.4 mm
- net BENDING_LIN_POT: track 139.8 -> 142.9 mm

Commit message: quick push with diode
Parts:
- added CR1: PMEG4010CEH, ${KIPRJMOD}:SOD123F_NXP, F.Cu at (199.9, 109.2)
Connections:
- U12 pad 22: GND -> (no net)
- U12 pad 23: GND -> (no net)
- U12 pad 24: GND -> (no net)
- U12 pad 25: GND -> (no net)
- U5 pad V: GND -> (no net)
Routing:
- net BENDING_LIN_POT: track 142.9 -> 187.2 mm, vias 2 -> 3
- net 3.3V: track 625.6 -> 630.8 mm
- net 5V: track 617.4 -> 618.8 mm
- net INDUCTIVE_PROX_2: track 126.3 -> 126.9 mm

Commit message: final connectors!
Connections:
- U12 pad 22: (no net) -> GND
- U12 pad 23: (no net) -> GND
- U12 pad 24: (no net) -> GND
- U12 pad 25: (no net) -> GND
- U5 pad V: (no net) -> GND
Routing:
- net GND: track 456.9 -> 479.9 mm
Changed lines of the file:
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@@
 			(layers "*.Cu" "*.Mask")
 			(remove_unused_layers no)
+			(net 2 "GND")
 		)
 		(pad "23" thru_hole circle
@@
 			(layers "*.Cu" "*.Mask")
 			(remove_unused_layers no)
+			(net 2 "GND")
 		)
 		(pad "24" thru_hole circle
@@
 			(layers "*.Cu" "*.Mask")
 			(remove_unused_layers no)
+			(net 2 "GND")
 		)
 		(pad "25" thru_hole circle
@@
 			(layers "*.Cu" "*.Mask")
 			(remove_unused_layers no)
+			(net 2 "GND")
 		)
 	)
@@
 			(layers "*.Cu" "*.Mask")
 			(remove_unused_layers no)
+			(net 2 "GND")
 		)
 		(pad "V" thru_hole circle
@@
 			(layers "*.Cu" "*.Mask")
 			(remove_unused_layers no)
+			(net 2 "GND")
 		)
 		(pad "V" thru_hole circle
@@
 			(layers "*.Cu" "*.Mask")
 			(remove_unused_layers no)
+			(net 2 "GND")
 		)
 	)
@@
 			(solder_mask_margin 0.102)
 		)
-		(pad "39_10" thru_hole circle
-			(at -2.2 -2.47 90)
-			(size 0.3 0.3)
-			(drill 0.2)
-			(layers "*.Cu" "*.Mask")
-			(remove_unused_layers no)
-			(net 2 "GND")
-			(pinfunction "GND")
-			(pintype "power_in")
-			(solder_mask_margin 0.102)
-		)
-		(pad "39_11" thru_hole circle
-			(at -0.8 -2.47 90)
-			(size 0.3 0.3)
-			(drill 0.2)
-			(layers "*.Cu" "*.Mask")
-			(remove_unused_layers no)
-			(net 2 "GND")
-			(pinfunction "GND")
-			(pintype "power_in")
-			(solder_mask_margin 0.102)
-		)
-		(pad "39_12" thru_hole circle
-			(at -2.9 -1.77 90)
-			(size 0.3 0.3)
-			(drill 0.2)
-			(layers "*.Cu" "*.Mask")
-			(remove_unused_layers no)
-			(net 2 "GND")
-			(pinfunction "GND")
-			(pintype "power_in")
-			(solder_mask_margin 0.102)
-		)
-		(pad "39_13" thru_hole circle
-			(at -1.5 -1.77 90)
-			(size 0.3 0.3)
-			(drill 0.2)
-			(layers "*.Cu" "*.Mask")
-			(remove_unused_layers no)
-			(net 2 "GND")
-			(pinfunction "GND")
-			(pintype "power_in")
-			(solder_mask_margin 0.102)
-		)
-		(pad "39_14" thru_hole circle
-			(at -0.1 -1.77 90)
-			(size 0.3 0.3)
-			(drill 0.2)
-			(layers "*.Cu" "*.Mask")
-			(remove_unused_layers no)
-			(net 2 "GND")
-			(pinfunction "GND")
-			(pintype "power_in")
-			(solder_mask_margin 0.102)
-		)
-		(pad "39_15" thru_hole circle
-			(at -2.2 -1.07 90)
-			(size 0.3 0.3)
-			(drill 0.2)
-			(layers "*.Cu" "*.Mask")
-			(remove_unused_layers no)
-			(net 2 "GND")
-			(pinfunction "GND")
-			(pintype "power_in")
-			(solder_mask_margin 0.102)
-		)
-		(pad "39_16" thru_hole circle
-			(at -0.8 -1.07 90)
-			(size 0.3 0.3)
-			(drill 0.2)
-			(layers "*.Cu" "*.Mask")
-			(remove_unused_layers no)
-			(net 2 "GND")
-			(pinfunction "GND")
-			(pintype "power_in")
-			(solder_mask_margin 0.102)
-		)
-		(pad "39_17" thru_hole circle
-			(at -2.9 -0.37 90)
-			(size 0.3 0.3)
-			(drill 0.2)
-			(layers "*.Cu" "*.Mask")
-			(remove_unused_layers no)
-			(net 2 "GND")
-			(pinfunction "GND")
-			(pintype "power_in")
-			(solder_mask_margin 0.102)
-		)
-		(pad "39_18" thru_hole circle
-			(at -1.5 -0.37 90)
-			(size 0.3 0.3)
-			(drill 0.2)
-			(layers "*.Cu" "*.Mask")
-			(remove_unused_layers no)
-			(net 2 "GND")
-			(pinfunction "GND")
-			(pintype "power_in")
-			(solder_mask_margin 0.102)
-		)
-		(pad "39_19" thru_hole circle
-			(at -0.1 -0.37 90)
-			(size 0.3 0.3)
-			(drill 0.2)
-			(layers "*.Cu" "*.Mask")
-			(remove_unused_layers no)
-			(net 2 "GND")
-			(pinfunction "GND")
-			(pintype "power_in")
-			(solder_mask_margin 0.102)
-		)
-		(pad "39_20" thru_hole circle
-			(at -2.2 0.33 90)
-			(size 0.3 0.3)
-			(drill 0.2)
-			(layers "*.Cu" "*.Mask")
-			(remove_unused_layers no)
-			(net 2 "GND")
-			(pinfunction "GND")
-			(pintype "power_in")
-			(solder_mask_margin 0.102)
-		)
-		(pad "39_21" thru_hole circle
-			(at -0.8 0.33 90)
-			(size 0.3 0.3)
-			(drill 0.2)
-			(layers "*.Cu" "*.Mask")
-			(remove_unused_layers no)
-			(net 2 "GND")
-			(pinfunction "GND")
-			(pintype "power_in")
-			(solder_mask_margin 0.102)
-		)
 	)
 	(footprint "Inductor_SMD:L_0805_2012Metric"
@@
 	)
 	(segment
+		(start 252.37125 129.735)
+		(end 252.37125 126.935)
+		(width 0.25)
+		(layer "F.Cu")
+		(net 2)
+	)
+	(segment
 		(start 75.824999 76.65)
 		(end 73.575 76.65)
@@
 	)
 	(segment
+		(start 250.97125 129.735)
+		(end 253.77125 129.735)
+		(width 0.25)
+		(layer "F.Cu")
+		(net 2)
+	)
+	(segment
 		(start 156.57449 91.5)
 		(end 158.97449 91.5)
@@
 	)
 	(segment
-		(start 250.97125 129.035)
-		(end 250.97125 128.335)
-		(width 0.25)
-		(layer "F.Cu")
-		(net 2)
-	)
-	(segment
 		(start 111.675 102.88)
 		(end 111.675 104.73)
@@
 	)
 	(segment
-		(start 75.499997 86.749997)
-		(end 75.5 86.75)
-		(width 0.25)
-		(layer "F.Cu")
-		(net 2)
-	)
-	(segment
 		(start 164.5 70.775)
 		(end 164.5 71.5)
@@
 	)
 	(segment
-		(start 250.97125 127.635)
-		(end 250.97125 126.935)
-		(width 0.25)
-		(layer "F.Cu")
-		(net 2)
-	)
-	(segment
 		(start 223.7 120.7)
 		(end 224.40475 120.7)
@@
 	)
 	(segment
-		(start 74.275001 86.749997)
-		(end 75.499997 86.749997)
-		(width 0.5)
-		(layer "F.Cu")
-		(net 2)
-	)
-	(segment
 		(start 159 71.5)
 		(end 159 70.1)
@@
 	)
 	(segment
+		(start 75.5 86.75)
+		(end 74.275004 86.75)
+		(width 0.25)
+		(layer "F.Cu")
+		(net 2)
+	)
+	(segment
 		(start 357.35 101.5746)
 		(end 357.35 100)
@@
 	)
 	(segment
+		(start 253.77125 129.735)
+		(end 253.77125 126.935)
+		(width 0.25)
+		(layer "F.Cu")
+		(net 2)
+	)
+	(segment
 		(start 130.75 192.6175)
 		(end 127 192.6175)
@@
 	)
 	(segment
+		(start 253.77125 126.935)
+		(end 250.97125 126.935)
+		(width 0.25)
+		(layer "F.Cu")
+		(net 2)
+	)
+	(segment
 		(start 74.6 192.6)
 		(end 71.65 192.6)
@@
 	)
 	(segment
+		(start 250.97125 126.935)
+		(end 250.97125 129.735)
+		(width 0.25)
+		(layer "F.Cu")
+		(net 2)
+	)
+	(segment
+		(start 250.97125 128.335)
+		(end 253.77125 128.335)
+		(width 0.25)
+		(layer "F.Cu")
+		(net 2)
+	)
+	(segment
 		(start 294.312236 143.28)
 		(end 294.312236 142.01)
@@
 	)
 	(segment
+		(start 249.88125 129.735)
+		(end 250.97125 129.735)
+		(width 0.25)
+		(layer "F.Cu")
+		(net 2)
+	)
+	(segment
 		(start 110.3 192.55)
 		(end 111.6 191.25)
@@
 	)
 	(segment
+		(start 245.03125 135.585)
+		(end 245.03125 134.585)
+		(width 0.25)
+		(layer "F.Cu")
+		(net 2)
+	)
+	(segment
 		(start 163 69.8)
 		(end 163.525 69.8)
@@
 	)
 	(segment
-		(start 250.97125 128.335)
-		(end 250.97125 127.635)
-		(width 0.25)
-		(layer "F.Cu")
-		(net 2)
-	)
-	(segment
 		(start 92.775 136.43)
 		(end 90.275 136.43)
@@
 	)
 	(segment
-		(start 250.97125 129.735)
-		(end 250.97125 129.035)
-		(width 0.25)
-		(layer "F.Cu")
-		(net 2)
-	)
-	(segment
 		(start 165.4 99.9875)
 		(end 164.7125 99.3)
@@
 	)
 	(segment
+		(start 245.03125 134.585)
+		(end 249.88125 129.735)
+		(width 0.25)
+		(layer "F.Cu")
+		(net 2)
+	)
+	(segment
 		(start 78.149999 88.349999)
 		(end 76.724999 88.349999)
@@
 		(layer "F.Cu")
 		(net 2)
+	)
+	(segment
+		(start 74.275004 86.75)
+		(end 74.275001 86.749997)
+		(width 0.25)
+		(layer "F.Cu")
+		(net 2)
