File: production/ecad/Tubender PCB/motors_actuators.kicad_sch (KiCad schematic)
At the start: 5 parts, among them J11 640387-8, J13 640387-5, J2 640387-5, J3 640387-5, J4 640387-5

Commit message: start power layout
Parts:
- J11: footprint 640387-8:TE_640387-8 -> ${KIPRJMOD}:TE_640387-8
- J13, J2, J3, J4: footprint 640387-5:TE_640387-5 -> ${KIPRJMOD}:TE_640387-5
Changed lines of the file:
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@@
 			)
 		)
-		(property "Footprint" "640387-5:TE_640387-5"
+		(property "Footprint" "${KIPRJMOD}:TE_640387-5"
 			(at 93.98 91.44 0)
 			(effects
@@
 			)
 		)
-		(property "Footprint" "640387-5:TE_640387-5"
+		(property "Footprint" "${KIPRJMOD}:TE_640387-5"
 			(at 226.06 91.44 0)
 			(effects
@@
 			)
 		)
-		(property "Footprint" "640387-5:TE_640387-5"
+		(property "Footprint" "${KIPRJMOD}:TE_640387-5"
 			(at 125.73 137.16 0)
 			(effects
@@
 			)
 		)
-		(property "Footprint" "640387-8:TE_640387-8"
+		(property "Footprint" "${KIPRJMOD}:TE_640387-8"
 			(at 196.85 138.43 0)
 			(effects
@@
 			)
 		)
-		(property "Footprint" "640387-5:TE_640387-5"
+		(property "Footprint" "${KIPRJMOD}:TE_640387-5"
 			(at 158.75 91.44 0)
 			(effects

Commit message: 0 Ohm Resistors
Added DNP 0 Ohm's connected to the 24V rail to the motor connectors power out pin. This is in case we have issues with the drivers taking 48 volts and to just have flexbility
Parts:
- added R76, R77, R78, R79, R80, R81, R82, R83: 0, Resistor_SMD:R_0805_2012Metric, symbol Device:R_US
Connections:
- net +48V: now also R77.2, R78.2, R80.2, R82.2; no longer J13.1, J2.1, J3.1, J4.1
- new net: J13.1, R82.1, R83.1
- new net: J2.1, R76.1, R77.1
- new net: J4.1, R80.1, R81.1
- new net: J3.1, R78.1, R79.1
- new net +24V: R76.2, R79.2, R81.2, R83.2
Other:
- moved on the sheet: J13
