File: production/ecad/Tubender PCB/sensors.kicad_sch (KiCad schematic)
At the start: 6 parts, among them J10 640387-5, J14 640387-3, J5 640387-6, J6 640387-6, J8 640387-6, J9 640387-5

Commit message: start power layout
Parts:
- J10, J9: footprint 640387-5:TE_640387-5 -> ${KIPRJMOD}:TE_640387-5
- J14: footprint 640387-3:TE_640387-3 -> ${KIPRJMOD}:TE_640387-3
- J5, J6, J8: footprint 640387-6:TE_640387-6 -> ${KIPRJMOD}:TE_640387-6
Changed lines of the file:
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@@
 			)
 		)
-		(property "Footprint" "640387-5:TE_640387-5"
+		(property "Footprint" "${KIPRJMOD}:TE_640387-5"
 			(at 203.2 93.98 0)
 			(effects
@@
 			)
 		)
-		(property "Footprint" "640387-3:TE_640387-3"
+		(property "Footprint" "${KIPRJMOD}:TE_640387-3"
 			(at 201.93 137.16 0)
 			(effects
@@
 			)
 		)
-		(property "Footprint" "640387-6:TE_640387-6"
+		(property "Footprint" "${KIPRJMOD}:TE_640387-6"
 			(at 128.27 138.43 0)
 			(effects
@@
 			)
 		)
-		(property "Footprint" "640387-5:TE_640387-5"
+		(property "Footprint" "${KIPRJMOD}:TE_640387-5"
 			(at 127 90.17 0)
 			(effects
@@
 			)
 		)
-		(property "Footprint" "640387-6:TE_640387-6"
+		(property "Footprint" "${KIPRJMOD}:TE_640387-6"
 			(at 203.2 52.07 0)
 			(effects
@@
 			)
 		)
-		(property "Footprint" "640387-6:TE_640387-6"
+		(property "Footprint" "${KIPRJMOD}:TE_640387-6"
 			(at 124.46 52.07 0)
 			(effects

Commit message: sensor updates!
Parts:
- removed J10, J9: 640387-5, ${KIPRJMOD}:TE_640387-5, symbol 640387-5:640387-5
- removed J5, J6, J8: 640387-6, ${KIPRJMOD}:TE_640387-6, symbol 640387-6:640387-6
- added J1, J10, J33, J34, J5, J6: 640387-2, 640387-2:TE_640387-2, symbol 640387-2:640387-2
- added J35, J37, J8, J9: 640387-3, ${KIPRJMOD}:TE_640387-3, symbol 640387-3:640387-3
- added R17, R6, R7, R8: 100k, Resistor_SMD:R_0805_2012Metric, symbol Device:R_Small_US
- added R18, R45: 10k, Resistor_SMD:R_0805_2012Metric, symbol Device:R_US
- added R43, R44, R71, R73: 5.1K, Resistor_SMD:R_0805_2012Metric, symbol Device:R_US
- added R48, R75: 0, Resistor_SMD:R_0805_2012Metric, symbol Device:R_US
- added R72, R74: 15k, Resistor_SMD:R_0805_2012Metric, symbol Device:R_US
Connections:
- net +12V: now also J8.1, J9.1, R48.2
- net +24V: now also R75.2; no longer J14.1
- net +5V: now also J10.1, J35.1, J37.1, J6.1, R43.2, R44.2
- net ADVANCE_LIMIT_1: now also J33.2, R8.2
- net ADVANCE_LIMIT_2: now also J34.2, R17.2
- net CHUCK_BEAM: now also J37.2, R44.1, R45.2
- net DIE_BEAM: now also J35.2, R18.2, R43.1
- net DIE_LIMIT_1: now also J1.2, R6.2
- net DIE_LIMIT_2: now also J5.2, R7.2
- net GND: now also J10.2, J35.3, J37.3, J6.2, J8.3, J9.3, R17.1, R18.1, R45.1, R6.1, R7.1, R71.1, R73.1, R8.1
- net INDUCTIVE_PROX_1: now also R71.2, R72.2
- net INDUCTIVE_PROX_2: now also R73.2, R74.2
- new net: J8.2, R74.1
- new net: J14.1, R48.1, R75.1
- new net: J9.2, R72.1
- new net +3.3V: J1.1, J33.1, J34.1, J5.1
Other:
- note added: "Advance Limit Switch Connectors"
- note added: "Chuck Break Beam Connectors"
- note added: "Die Break Beam Connectors"
- note added: "Die Limit Switch Connectors"
- note removed: "Advance Limit Switch Connector"
- note removed: "Chuck Break Beam Connector"
- note removed: "Die Break Beam Connector"
- note removed: "Die Limit Switch Connector"
- moved on the sheet: J14

Commit message: working on mcu layout
Parts:
- J1, J10, J33, J34, J5, J6: footprint 640387-2:TE_640387-2 -> ${KIPRJMOD}:TE_640387-2
Changed lines of the file:
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@@
 			)
 		)
-		(property "Footprint" "640387-2:TE_640387-2"
+		(property "Footprint" "${KIPRJMOD}:TE_640387-2"
 			(at 80.01 43.18 0)
 			(effects
@@
 			)
 		)
-		(property "Footprint" "640387-2:TE_640387-2"
+		(property "Footprint" "${KIPRJMOD}:TE_640387-2"
 			(at 156.21 43.18 0)
 			(effects
@@
 			)
 		)
-		(property "Footprint" "640387-2:TE_640387-2"
+		(property "Footprint" "${KIPRJMOD}:TE_640387-2"
 			(at 73.66 99.06 0)
 			(effects
@@
 			)
 		)
-		(property "Footprint" "640387-2:TE_640387-2"
+		(property "Footprint" "${KIPRJMOD}:TE_640387-2"
 			(at 152.4 99.06 0)
 			(effects
@@
 			)
 		)
-		(property "Footprint" "640387-2:TE_640387-2"
+		(property "Footprint" "${KIPRJMOD}:TE_640387-2"
 			(at 156.21 59.69 0)
 			(effects
@@
 			)
 		)
-		(property "Footprint" "640387-2:TE_640387-2"
+		(property "Footprint" "${KIPRJMOD}:TE_640387-2"
 			(at 80.01 59.69 0)
 			(effects

Commit message: Potentiometer Update
Parts:
- added R84: 15k, Resistor_SMD:R_0805_2012Metric, symbol Device:R_US
- R75: now not fitted; now left out of the parts list
Connections:
- net BENDING_LIN_POT: now also R84.1
- net at J14.1, R48.1, R75.1: now also R84.2
Other:
- moved on the sheet: R48
Changed lines of the file:
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@@
 	)
 	(junction
-		(at 58.42 110.49)
+		(at 215.9 53.34)
 		(diameter 0)
 		(color 0 0 0 0)
 	)
 	(junction
-		(at 63.5 43.18)
+		(at 58.42 110.49)
 		(diameter 0)
 		(color 0 0 0 0)
 	)
 	(junction
-		(at 227.33 129.54)
+		(at 63.5 43.18)
 		(diameter 0)
 		(color 0 0 0 0)
 	)
 	(junction
-		(at 137.16 110.49)
+		(at 227.33 129.54)
 		(diameter 0)
 		(color 0 0 0 0)
 	)
 	(junction
-		(at 220.98 53.34)
+		(at 137.16 110.49)
 		(diameter 0)
 		(color 0 0 0 0)
@@
 	)
 	(junction
+		(at 218.44 63.5)
+		(diameter 0)
+		(color 0 0 0 0)
+	)
+	(junction
 		(at 139.7 43.18)
 		(diameter 0)
@@
 	)
 	(junction
+		(at 218.44 53.34)
+		(diameter 0)
+		(color 0 0 0 0)
+	)
+	(junction
 		(at 63.5 59.69)
 		(diameter 0)
@@
 	(wire
 		(pts
-			(xy 207.01 53.34) (xy 220.98 53.34)
+			(xy 207.01 53.34) (xy 215.9 53.34)
+		)
+		(stroke
+			(width 0)
+			(type default)
+		)
+	)
+	(wire
+		(pts
+			(xy 215.9 53.34) (xy 218.44 53.34)
 		)
 		(stroke
@@
 	(wire
 		(pts
-			(xy 218.44 55.88) (xy 226.06 55.88)
+			(xy 215.9 63.5) (xy 218.44 63.5)
 		)
 		(stroke
@@
 	(wire
 		(pts
+			(xy 218.44 60.96) (xy 218.44 63.5)
+		)
+		(stroke
+			(width 0)
+			(type default)
+		)
+	)
+	(wire
+		(pts
 			(xy 146.05 57.15) (xy 130.81 57.15)
 		)
@@
 	(wire
 		(pts
+			(xy 220.98 63.5) (xy 220.98 55.88)
+		)
+		(stroke
+			(width 0)
+			(type default)
+		)
+	)
+	(wire
+		(pts
 			(xy 139.7 59.69) (xy 146.05 59.69)
 		)
@@
 	(wire
 		(pts
-			(xy 220.98 53.34) (xy 226.06 53.34)
-		)
-		(stroke
-			(width 0)
-			(type default)
-		)
-	)
-	(wire
-		(pts
 			(xy 50.8 96.52) (xy 63.5 96.52)
 		)
@@
 	(wire
 		(pts
+			(xy 218.44 63.5) (xy 220.98 63.5)
+		)
+		(stroke
+			(width 0)
+			(type default)
+		)
+	)
+	(wire
+		(pts
+			(xy 220.98 55.88) (xy 226.06 55.88)
+		)
+		(stroke
+			(width 0)
+			(type default)
+		)
+	)
+	(wire
+		(pts
 			(xy 50.8 100.33) (xy 50.8 99.06)
 		)
@@
 		)
 	)
+	(wire
+		(pts
+			(xy 218.44 53.34) (xy 226.06 53.34)
+		)
+		(stroke
+			(width 0)
+			(type default)
+		)
+	)
 	(rectangle
 		(start 193.04 88.9)
@@
 	(global_label "BENDING_LIN_POT"
 		(shape input)
-		(at 218.44 55.88 180)
+		(at 215.9 63.5 180)
 		(fields_autoplaced yes)
 		(effects
@@
 		)
 		(property "Intersheetrefs" "${INTERSHEET_REFS}"
-			(at 198.7633 55.88 0)
+			(at 196.2233 63.5 0)
 			(effects
 				(font
@@
 	)
 	(symbol
+		(lib_id "Device:R_US")
+		(at 218.44 57.15 0)
+		(mirror x)
+		(unit 1)
+		(exclude_from_sim no)
+		(in_bom yes)
+		(on_board yes)
+		(dnp no)
+		(property "Reference" "R84"
+			(at 212.852 57.15 90)
+			(effects
+				(font
+					(size 1.27 1.27)
+				)
+			)
+		)
+		(property "Value" "15k"
+			(at 215.138 56.896 90)
+			(effects
+				(font
+					(size 1.27 1.27)
+				)
+			)
+		)
+		(property "Footprint" "Resistor_SMD:R_0805_2012Metric"
+			(at 219.456 56.896 90)
+			(effects
+				(font
+					(size 1.27 1.27)
+				)
+				(hide yes)
+			)
+		)
+		(property "Datasheet" "~"
+			(at 218.44 57.15 0)
+			(effects
+				(font
+					(size 1.27 1.27)
+				)
+				(hide yes)
+			)
+		)
+		(property "Description" "Resistor, US symbol"
+			(at 218.44 57.15 0)
+			(effects
+				(font
+					(size 1.27 1.27)
+				)
+				(hide yes)
+			)
+		)
+		(pin "2"
+		)
+		(pin "1"
+		)
+		(instances
+			(project "Tubender PCB"
+				(path "/3e1aedd0-6089-4edb-92c7-0c31da2e7927/cace885d-07c2-48b7-a983-3b69a09d8a62"
+					(reference "R84")
+					(unit 1)
+				)
+			)
+		)
+	)
+	(symbol
 		(lib_id "640387-3:640387-3")
 		(at 237.49 121.92 0)
@@
 	(symbol
 		(lib_id "power:+24V")
-		(at 220.98 45.72 0)
+		(at 215.9 45.72 0)
 		(unit 1)
 		(exclude_from_sim no)
@@
 		(dnp no)
 		(property "Reference" "#PWR098"
-			(at 220.98 49.53 0)
+			(at 215.9 49.53 0)
 			(effects
 				(font
@@
 		)
 		(property "Value" "+12V"
-			(at 220.726 41.91 0)
+			(at 215.646 41.91 0)
 			(effects
 				(font
@@
 		)
 		(property "Footprint" ""
-			(at 220.98 45.72 0)
+			(at 215.9 45.72 0)
 			(effects
 				(font
@@
 		)
 		(property "Datasheet" ""
-			(at 220.98 45.72 0)
+			(at 215.9 45.72 0)
 			(effects
 				(font
@@
 		)
 		(property "Description" "Power symbol creates a global label with name \"+24V\""
-			(at 220.98 45.72 0)
+			(at 215.9 45.72 0)
 			(effects
 				(font
@@
 	(symbol
 		(lib_id "Device:R_US")
-		(at 220.98 49.53 0)
+		(at 215.9 49.53 0)
 		(mirror x)
 		(unit 1)
@@
 		(dnp no)
 		(property "Reference" "R48"
-			(at 218.186 49.53 90)
+			(at 213.106 49.53 90)
 			(effects
 				(font
@@
 		)
 		(property "Value" "0"
-			(at 224.79 49.53 90)
+			(at 219.71 49.53 90)
 			(effects
 				(font
@@
 		)
 		(property "Footprint" "Resistor_SMD:R_0805_2012Metric"
-			(at 221.996 49.276 90)
+			(at 216.916 49.276 90)
 			(effects
 				(font
@@
 		)
 		(property "Datasheet" "~"
-			(at 220.98 49.53 0)
+			(at 215.9 49.53 0)
 			(effects
 				(font
@@
 		)
 		(property "Description" "Resistor, US symbol"
-			(at 220.98 49.53 0)
+			(at 215.9 49.53 0)
 			(effects
 				(font
@@
 		(unit 1)
 		(exclude_from_sim no)
-		(in_bom yes)
+		(in_bom no)
 		(on_board yes)
-		(dnp no)
+		(dnp yes)
 		(property "Reference" "R75"
 			(at 204.216 49.53 90)
