File: production/ecad/Tubender PCB/control.kicad_sch (KiCad schematic)
At the start: 52 parts, among them J32 USB4110GFA, Q1 AO3400A, Q2 AO3400A, U10 MCP23017-E_SO, U2 ESP32-WROOM-32UE_M113EH6400UH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, U3 MCP23017-E_SO, U6 CP2102N-A02-GQFN28

Commit message: minor changes and vias
Connections:
- net at C10.1, D13.2, J32.A7 (DN1)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: no longer C11.1, D14.2, J32.A6 (DP1), J32.B6 (DP2), U6.4 (D+)
- new net: C11.1, D14.2, J32.A6 (DP1), J32.B6 (DP2), U6.4 (D+)
Changed lines of the file:
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@@
-	)
-	(junction
-		(at 167.64 80.01)
-		(diameter 0)
-		(color 0 0 0 0)
 	)
 	(junction
@@
 	(wire
 		(pts
-			(xy 167.64 80.01) (xy 213.36 80.01)
+			(xy 158.75 80.01) (xy 213.36 80.01)
 		)
 		(stroke
@@
 		)
 		(stroke
-			(width 0)
-			(type default)
-		)
-	)
-	(wire
-		(pts
-			(xy 158.75 80.01) (xy 167.64 80.01)
-		)
-		(stroke

Commit message: Fixed MCU Pinout Schematic
Parts:
- R19, R4: value 1K -> 4.7k
- R68: value 1k -> 4.7k
Connections:
- net ADVANCING_ENA+: now also U10.8 (GPB7); no longer U2.27 (IO16)
- net BENDING_LIN_POT: now also U2.7 (IO35); no longer U10.1 (GPB0)
- net BENDING_LPWM: now also U2.27 (IO16); no longer U10.8 (GPB7)
- net BENDING_RPWM: now also U2.16 (IO13); no longer U10.6 (GPB5)
- net CHUCK_CLAMP_ENA+: now also U2.10 (IO25); no longer U2.8 (IO32)
- net DIE_CLAMP_ENA+: now also U10.6 (GPB5); no longer U2.16 (IO13)
- net ROTATION_ENA+: now also U10.1 (GPB0); no longer U2.10 (IO25)
- no-connect marks 25 -> 24

Commit message: More MCU Updates
Connections:
- net 7-SEG_OEb: now also U10.26 (GPA5); no longer U10.27 (GPA6)
- net 7-SEG_RCLK: now also U2.8 (IO32); no longer U10.26 (GPA5)
- net 7-SEG_SER: now also U2.10 (IO25); no longer U10.24 (GPA3)
- net 7-SEG_SRCLK: now also U2.11 (IO26); no longer U10.25 (GPA4)
- net BENDING_L_ENA: now also U10.27 (GPA6); no longer U10.28 (GPA7)
- net CHUCK_CLAMP_ENA+: now also U10.25 (GPA4); no longer U2.10 (IO25)
- net CHUCK_CLAMP_PUL+: now also U10.24 (GPA3); no longer U2.12 (IO27)
- net ROTATION_DIR+: now also U2.12 (IO27); no longer U2.11 (IO26)
- no-connect marks 24 -> 25
Changed lines of the file:
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@@
 	)
 	(no_connect
+		(at 363.22 127)
+	)
+	(no_connect
 		(at 213.36 100.33)
 	)
@@
 	(wire
 		(pts
-			(xy 365.76 127) (xy 363.22 127)
-		)
-		(stroke
-			(width 0)
-			(type default)
-		)
-	)
-	(wire
-		(pts
 			(xy 318.77 106.68) (xy 320.04 106.68)
 		)
@@
 		)
 	)
+	(global_label "7-SEG_SRCLK"
+		(shape input)
+		(at 153.67 210.82 0)
+		(fields_autoplaced yes)
+		(effects
+			(font
+				(size 1.27 1.27)
+			)
+			(justify left)
+		)
+		(property "Intersheetrefs" "${INTERSHEET_REFS}"
+			(at 170.0808 210.82 0)
+			(effects
+				(font
+					(size 1.27 1.27)
+				)
+				(justify left)
+				(hide yes)
+			)
+		)
+	)
 	(global_label "DIE_CLAMP_PUL+"
 		(shape input)
@@
 		)
 	)
+	(global_label "7-SEG_RCLK"
+		(shape input)
+		(at 153.67 215.9 0)
+		(fields_autoplaced yes)
+		(effects
+			(font
+				(size 1.27 1.27)
+			)
+			(justify left)
+		)
+		(property "Intersheetrefs" "${INTERSHEET_REFS}"
+			(at 168.8713 215.9 0)
+			(effects
+				(font
+					(size 1.27 1.27)
+				)
+				(justify left)
+				(hide yes)
+			)
+		)
+	)
 	(global_label "DIE_LIMIT_2"
 		(shape input)
@@
 		)
 	)
-	(global_label "CHUCK_CLAMP_PUL+"
-		(shape input)
-		(at 153.67 213.36 0)
-		(fields_autoplaced yes)
-		(effects
-			(font
-				(size 1.27 1.27)
-			)
-			(justify left)
-		)
-		(property "Intersheetrefs" "${INTERSHEET_REFS}"
-			(at 176.3705 213.36 0)
-			(effects
-				(font
-					(size 1.27 1.27)
-				)
-				(justify left)
-				(hide yes)
-			)
-		)
-	)
 	(global_label "DISPLAY_MISO"
 		(shape input)
@@
 		)
 	)
+	(global_label "ROTATION_DIR+"
+		(shape input)
+		(at 153.67 213.36 0)
+		(fields_autoplaced yes)
+		(effects
+			(font
+				(size 1.27 1.27)
+			)
+			(justify left)
+		)
+		(property "Intersheetrefs" "${INTERSHEET_REFS}"
+			(at 171.2301 213.36 0)
+			(effects
+				(font
+					(size 1.27 1.27)
+				)
+				(justify left)
+				(hide yes)
+			)
+		)
+	)
 	(global_label "7-SEG_SER"
 		(shape input)
@@
 		)
 	)
-	(global_label "ROTATION_DIR+"
-		(shape input)
-		(at 153.67 210.82 0)
-		(fields_autoplaced yes)
-		(effects
-			(font
-				(size 1.27 1.27)
-			)
-			(justify left)
-		)
-		(property "Intersheetrefs" "${INTERSHEET_REFS}"
-			(at 171.2301 210.82 0)
-			(effects
-				(font
-					(size 1.27 1.27)
-				)
-				(justify left)
-				(hide yes)
-			)
-		)
-	)
 	(global_label "BUTTON_CHAN_SEL_2A"
 		(shape input)
@@
 	(global_label "BENDING_L_ENA"
 		(shape input)
-		(at 365.76 127 0)
-		(fields_autoplaced yes)
-		(effects
-			(font
-				(size 1.27 1.27)
-			)
-			(justify left)
-		)
-		(property "Intersheetrefs" "${INTERSHEET_REFS}"
-			(at 383.5014 127 0)
-			(effects
-				(font
-					(size 1.27 1.27)
-				)
-				(justify left)
-				(hide yes)
-			)
-		)
-	)
-	(global_label "BENDING_L_ENA"
-		(shape input)
 		(at 44.45 110.49 180)
 		(fields_autoplaced yes)
@@
 		)
 	)
-	(global_label "7-SEG_OEb"
-		(shape input)
-		(at 365.76 124.46 0)
-		(fields_autoplaced yes)
-		(effects
-			(font
-				(size 1.27 1.27)
-			)
-			(justify left)
-		)
-		(property "Intersheetrefs" "${INTERSHEET_REFS}"
-			(at 379.7517 124.46 0)
-			(effects
-				(font
-					(size 1.27 1.27)
-				)
-				(justify left)
-				(hide yes)
-			)
-		)
-	)
 	(global_label "BUTTON_PLEX_2"
 		(shape input)
@@
 		)
 	)
+	(global_label "7-SEG_OEb"
+		(shape input)
+		(at 365.76 121.92 0)
+		(fields_autoplaced yes)
+		(effects
+			(font
+				(size 1.27 1.27)
+			)
+			(justify left)
+		)
+		(property "Intersheetrefs" "${INTERSHEET_REFS}"
+			(at 379.7517 121.92 0)
+			(effects
+				(font
+					(size 1.27 1.27)
+				)
+				(justify left)
+				(hide yes)
+			)
+		)
+	)
 	(global_label "ADVANCE_LIMIT_2"
 		(shape input)
@@
 		)
 	)
-	(global_label "7-SEG_SER"
+	(global_label "CHUCK_CLAMP_PUL+"
 		(shape input)
 		(at 365.76 116.84 0)
@@
 		)
 		(property "Intersheetrefs" "${INTERSHEET_REFS}"
-			(at 379.7517 116.84 0)
+			(at 388.4605 116.84 0)
 			(effects
 				(font
@@
 		)
 	)
+	(global_label "CHUCK_CLAMP_ENA+"
+		(shape input)
+		(at 365.76 119.38 0)
+		(fields_autoplaced yes)
+		(effects
+			(font
+				(size 1.27 1.27)
+			)
+			(justify left)
+		)
+		(property "Intersheetrefs" "${INTERSHEET_REFS}"
+			(at 388.4 119.38 0)
+			(effects
+				(font
+					(size 1.27 1.27)
+				)
+				(justify left)
+				(hide yes)
+			)
+		)
+	)
 	(global_label "DIE_CLAMP_PUL+"
 		(shape input)
@@
 		)
 	)
-	(global_label "7-SEG_RCLK"
+	(global_label "ESP_EN"
 		(shape input)
-		(at 365.76 121.92 0)
+		(at 100.33 170.18 180)
 		(fields_autoplaced yes)
 		(effects
@@
 				(size 1.27 1.27)
 			)
-			(justify left)
+			(justify right)
 		)
 		(property "Intersheetrefs" "${INTERSHEET_REFS}"
-			(at 380.9613 121.92 0)
+			(at 90.2692 170.18 0)
 			(effects
 				(font
 					(size 1.27 1.27)
 				)
-				(justify left)
+				(justify right)
 				(hide yes)
 			)
 		)
 	)
-	(global_label "ESP_EN"
+	(global_label "7-SEG_SER"
 		(shape input)
-		(at 100.33 170.18 180)
+		(at 153.67 208.28 0)
 		(fields_autoplaced yes)
 		(effects
@@
 				(size 1.27 1.27)
 			)
-			(justify right)
+			(justify left)
 		)
 		(property "Intersheetrefs" "${INTERSHEET_REFS}"
-			(at 90.2692 170.18 0)
+			(at 167.6617 208.28 0)
 			(effects
 				(font
 					(size 1.27 1.27)
 				)
-				(justify right)
+				(justify left)
 				(hide yes)
 			)
@@
 		)
 	)
-	(global_label "CHUCK_CLAMP_ENA+"
-		(shape input)
-		(at 153.67 208.28 0)
-		(fields_autoplaced yes)
-		(effects
-			(font
-				(size 1.27 1.27)
-			)
-			(justify left)
-		)
-		(property "Intersheetrefs" "${INTERSHEET_REFS}"
-			(at 176.31 208.28 0)
-			(effects
-				(font
-					(size 1.27 1.27)
-				)
-				(justify left)
-				(hide yes)
-			)
-		)
-	)
 	(global_label "BENDING_R_ENA"
 		(shape input)
@@
 		)
 	)
-	(global_label "7-SEG_SRCLK"
-		(shape input)
-		(at 365.76 119.38 0)
-		(fields_autoplaced yes)
-		(effects
-			(font
-				(size 1.27 1.27)
-			)
-			(justify left)
-		)
-		(property "Intersheetrefs" "${INTERSHEET_REFS}"
-			(at 382.1708 119.38 0)
-			(effects
-				(font
-					(size 1.27 1.27)
-				)
-				(justify left)
-				(hide yes)
-			)
-		)
-	)
 	(global_label "DIE_LIMIT_2"
 		(shape input)
@@
 				(hide yes)
 			)
+		)
+	)
+	(global_label "BENDING_L_ENA"
+		(shape input)
+		(at 365.76 124.46 0)
+		(fields_autoplaced yes)
+		(effects
+			(font
+				(size 1.27 1.27)
+			)
+			(justify left)
+		)
+		(property "Intersheetrefs" "${INTERSHEET_REFS}"
+			(at 383.5014 124.46 0)
+			(effects
+				(font
+					(size 1.27 1.27)
+				)
+				(justify left)
+				(hide yes)
+			)

Commit message: Updated Layout for new MCU Connections
Connections:
- net 7-SEG_OEb: now also U10.24 (GPA3); no longer U10.26 (GPA5)
- net 7-SEG_RCLK: now also U2.12 (IO27); no longer U2.8 (IO32)
- net ADVANCING_PUL+: now also U2.27 (IO16); no longer U2.23 (IO15)
- net BENDING_LPWM: now also U2.23 (IO15); no longer U2.27 (IO16)
- net BENDING_RPWM: now also U2.13 (IO14); no longer U2.16 (IO13)
- net BENDING_R_ENA: now also U10.28 (GPA7); no longer U10.7 (GPB6)
- net CHUCK_CLAMP_DIR+: now also U2.26 (IO4); no longer U2.9 (IO33)
- net CHUCK_CLAMP_PUL+: now also U10.26 (GPA5); no longer U10.24 (GPA3)
- net DIE_CLAMP_DIR+: now also U2.16 (IO13); no longer U2.13 (IO14)
- net ROTATION_DIR+: now also U2.8 (IO32); no longer U2.12 (IO27)
- net ROTATION_ENA+: now also U10.7 (GPB6); no longer U10.1 (GPB0)
- net ROTATION_PUL+: now also U2.9 (IO33); no longer U2.26 (IO4)

Commit message: Differential Pairs
Connections:
- net USB_DN: now reaches C10.1, D13.2, J32.A7 (DN1), J32.B7 (DN2), U6.5 (D-)
- net USB_DP: now reaches C11.1, D14.2, J32.A6 (DP1), J32.B6 (DP2), U6.4 (D+)
Changed lines of the file:
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@@
+		)
+	)
+	(label "USB_DP"
+		(at 138.43 71.12 0)
+		(fields_autoplaced yes)
+		(effects
+			(font
+				(size 1.27 1.27)
+			)
+			(justify left bottom)
+		)
+	)
+	(label "USB_DN"
+		(at 177.8 80.01 0)
+		(fields_autoplaced yes)
+		(effects
+			(font
+				(size 1.27 1.27)
+			)
+			(justify left bottom)
 		)
 	)

Commit message: Potentiometer Update
Parts:
- added CR1: PMEG4010CEH, footprints:SOD123F_NXP, symbol 2024-11-01_00-41-16:PMEG4010CEH
Connections:
- net +3.3V: now also CR1.1
- net BENDING_LIN_POT: now also CR1.2
Changed lines of the file:
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@@
 	)
 	(junction
+		(at 99.06 213.36)
+		(diameter 0)
+		(color 0 0 0 0)
+	)
+	(junction
 		(at 167.64 77.47)
 		(diameter 0)
@@
 	(wire
 		(pts
+			(xy 101.6 200.66) (xy 101.6 213.36)
+		)
+		(stroke
+			(width 0)
+			(type default)
+		)
+	)
+	(wire
+		(pts
 			(xy 147.32 215.9) (xy 153.67 215.9)
 		)
@@
 	(wire
 		(pts
+			(xy 99.06 213.36) (xy 101.6 213.36)
+		)
+		(stroke
+			(width 0)
+			(type default)
+		)
+	)
+	(wire
+		(pts
 			(xy 317.5 226.06) (xy 317.5 228.6)
 		)
@@
 	(wire
 		(pts
-			(xy 105.41 200.66) (xy 106.68 200.66)
-		)
-		(stroke
-			(width 0)
-			(type default)
-		)
-	)
-	(wire
-		(pts
 			(xy 157.48 76.2) (xy 157.48 80.01)
 		)
@@
 	(wire
 		(pts
+			(xy 97.79 213.36) (xy 99.06 213.36)
+		)
+		(stroke
+			(width 0)
+			(type default)
+		)
+	)
+	(wire
+		(pts
 			(xy 52.07 133.35) (xy 44.45 133.35)
 		)
@@
 	(wire
 		(pts
+			(xy 106.68 200.66) (xy 101.6 200.66)
+		)
+		(stroke
+			(width 0)
+			(type default)
+		)
+	)
+	(wire
+		(pts
 			(xy 52.07 151.13) (xy 44.45 151.13)
 		)
@@
 	)
 	(rectangle
-		(start 85.09 143.51)
+		(start 77.47 143.51)
 		(end 199.39 241.3)
 		(stroke
@@
 	(text "ESP32"
 		(exclude_from_sim no)
-		(at 90.678 141.732 0)
+		(at 83.82 141.986 0)
 		(effects
 			(font
@@
 	(global_label "BENDING_LIN_POT"
 		(shape input)
-		(at 105.41 200.66 180)
+		(at 97.79 213.36 180)
 		(fields_autoplaced yes)
 		(effects
@@
 		)
 		(property "Intersheetrefs" "${INTERSHEET_REFS}"
-			(at 85.7333 200.66 0)
+			(at 78.1133 213.36 0)
 			(effects
 				(font
@@
 	)
 	(symbol
+		(lib_id "power:+24V")
+		(at 99.06 203.2 0)
+		(unit 1)
+		(exclude_from_sim no)
+		(in_bom yes)
+		(on_board yes)
+		(dnp no)
+		(property "Reference" "#PWR0219"
+			(at 99.06 207.01 0)
+			(effects
+				(font
+					(size 1.27 1.27)
+				)
+				(hide yes)
+			)
+		)
+		(property "Value" "+3.3V"
+			(at 99.06 199.136 0)
+			(effects
+				(font
+					(size 1.27 1.27)
+				)
+			)
+		)
+		(property "Footprint" ""
+			(at 99.06 203.2 0)
+			(effects
+				(font
+					(size 1.27 1.27)
+				)
+				(hide yes)
+			)
+		)
+		(property "Datasheet" ""
+			(at 99.06 203.2 0)
+			(effects
+				(font
+					(size 1.27 1.27)
+				)
+				(hide yes)
+			)
+		)
+		(property "Description" "Power symbol creates a global label with name \"+24V\""
+			(at 99.06 203.2 0)
+			(effects
+				(font
+					(size 1.27 1.27)
+				)
+				(hide yes)
+			)
+		)
+		(pin "1"
+		)
+		(instances
+			(project "Tubender PCB"
+				(path "/3e1aedd0-6089-4edb-92c7-0c31da2e7927/970b1c80-6c89-48ca-aa97-a5b3735d13b7"
+					(reference "#PWR0219")
+					(unit 1)
+				)
+			)
+		)
+	)
+	(symbol
 		(lib_id "Device:R_US")
 		(at 212.09 55.88 180)
@@
 					(unit 1)
 				)
+			)
+		)
+	)
+	(symbol
+		(lib_id "2024-11-01_00-41-16:PMEG4010CEH")
+		(at 99.06 213.36 90)
+		(unit 1)
+		(exclude_from_sim no)
+		(in_bom yes)
+		(on_board yes)
+		(dnp no)
+		(property "Reference" "CR1"
+			(at 102.108 208.026 90)
+			(effects
+				(font
+					(size 1.524 1.524)
+				)
+				(justify right)
+			)
+		)
+		(property "Value" "PMEG4010CEH"
+			(at 78.74 208.026 90)
+			(effects
+				(font
+					(size 1.524 1.524)
+				)
+				(justify right)
+				(hide yes)
+			)
+		)
+		(property "Footprint" "footprints:SOD123F_NXP"
+			(at 99.06 213.36 0)
+			(effects
+				(font
+					(size 1.27 1.27)
+					(italic yes)
+				)
+				(hide yes)
+			)
+		)
+		(property "Datasheet" "PMEG4010CEH"
+			(at 99.06 213.36 0)
+			(effects
+				(font
+					(size 1.27 1.27)
+					(italic yes)
+				)
+				(hide yes)
+			)
+		)
+		(property "Description" ""
+			(at 99.06 213.36 0)
+			(effects
+				(font
+					(size 1.27 1.27)
+				)
+				(hide yes)
+			)
+		)
+		(pin "1"
+		)
+		(pin "2"
+		)
+		(instances
+			(project ""
+				(path "/3e1aedd0-6089-4edb-92c7-0c31da2e7927/970b1c80-6c89-48ca-aa97-a5b3735d13b7"
+					(reference "CR1")
+					(unit 1)
+				)

Commit message: quick push with diode
Parts:
- CR1: footprint footprints:SOD123F_NXP -> ${KIPRJMOD}:SOD123F_NXP
Changed lines of the file:
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@@
 			)
 		)
-		(property "Footprint" "footprints:SOD123F_NXP"
+		(property "Footprint" "${KIPRJMOD}:SOD123F_NXP"
 			(at 99.06 213.36 0)
 			(effects

Commit message: DRC and INTA
Fixed the final DRC issue and also attached the interupt pin from the expander with lots of our sensors to the ESP
Connections:
- net INT_A: now reaches U2.6 (IO34)
- net INT_A: now also U3.20 (INTA)
- no-connect marks 25 -> 23
Changed lines of the file:
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@@
 	)
 	(no_connect
-		(at 106.68 198.12)
-	)
-	(no_connect
 		(at 259.08 74.93)
 	)
@@
 	)
 	(no_connect
-		(at 364.49 80.01)
-	)
-	(no_connect
 		(at 101.6 81.28)
 	)
@@
 	(wire
 		(pts
+			(xy 377.19 80.01) (xy 364.49 80.01)
+		)
+		(stroke
+			(width 0)
+			(type default)
+		)
+	)
+	(wire
+		(pts
 			(xy 260.35 115.57) (xy 260.35 113.03)
 		)
@@
 	(wire
 		(pts
+			(xy 86.36 198.12) (xy 106.68 198.12)
+		)
+		(stroke
+			(width 0)
+			(type default)
+		)
+	)
+	(wire
+		(pts
 			(xy 52.07 62.23) (xy 44.45 62.23)
 		)
@@
 		)
 	)
+	(global_label "INT_A"
+		(shape input)
+		(at 86.36 198.12 180)
+		(fields_autoplaced yes)
+		(effects
+			(font
+				(size 1.27 1.27)
+			)
+			(justify right)
+		)
+		(property "Intersheetrefs" "${INTERSHEET_REFS}"
+			(at 78.4157 198.12 0)
+			(effects
+				(font
+					(size 1.27 1.27)
+				)
+				(justify right)
+				(hide yes)
+			)
+		)
+	)
 	(global_label "ESP_RXD"
 		(shape input)
@@
 				(hide yes)
 			)
+		)
+	)
+	(global_label "INT_A"
+		(shape input)
+		(at 377.19 80.01 0)
+		(fields_autoplaced yes)
+		(effects
+			(font
+				(size 1.27 1.27)
+			)
+			(justify left)
+		)
+		(property "Intersheetrefs" "${INTERSHEET_REFS}"
+			(at 385.1343 80.01 0)
+			(effects
+				(font
+					(size 1.27 1.27)
+				)
+				(justify left)
+				(hide yes)
+			)
