File: production/ecad/Tubender Main_PCB/motors_actuators.kicad_sch (KiCad schematic)
At the start: 5 parts, among them J11 640387-8, J13 640387-5, J2 640387-5, J3 640387-5, J4 640387-5

Commit message: Fixed the Nets
Connections:
- net 12V renamed +12V
- net 5V renamed +5V
Other:
- note added: "Inputs"
- note added: "Power"
- moved on the sheet: J11, J13, J2, J3, J4
