File: production/ecad/Tubender UI_PCB/_autosave-user_interface.kicad_sch (KiCad schematic)
At the start: 16 parts, among them IC3 SN74LVC1G29DCTR, J1 640387-5, J2 1-640387-0, J3 104031-0811, U5 74HC595, U6 PEC11R-4215K-S0024

Commit message: Added UI footprints and first draft of layout
Parts:
- added J4: 640387-5, footprints:TE_640387-5, symbol 640387-5:640387-5
Connections:
- net +3V3: now also J4.5
- net SD_CD: now also J4.2
- net SD_CLK: now also J4.1
- net SD_CMD: now also J4.3
- net SD_DAT0: now also J4.4
Other:
- note added: "SD CARD"
- note added: "SD CARD Connector"
